Commit message: use package:// instead of file://

File: urdf/intel_realsense_d435.urdf.xacro (robot description, xacro)
@@ -65,5 +65,5 @@
         <origin xyz="0.0 0.0 0.0" rpy="0.0 0.0 0.0" />
         <geometry>
-          <mesh filename="file://$(find ros_components_description)/meshes/intel_realsense_d435.dae" />
+          <mesh filename="package://ros_components_description/meshes/intel_realsense_d435.dae" />
         </geometry>
       </visual>

File: urdf/orbbec_astra.urdf.xacro (robot description, xacro)
@@ -22,5 +22,5 @@
         <origin xyz="0.0 0.0 0.0" rpy="0.0 0.0 0.0" />
         <geometry>
-          <mesh filename="file://$(find ros_components_description)/meshes/orbbec_astra.dae" />
+          <mesh filename="package://ros_components_description/meshes/orbbec_astra.dae" />
         </geometry>
       </visual>

File: urdf/ouster_os1_32.urdf.xacro (robot description, xacro)
@@ -31,5 +31,5 @@
         <origin xyz="0.0 0.0 0.0" rpy="0.0 0.0 0.0" />
         <geometry>
-          <mesh filename="file://$(find ros_components_description)/meshes/ouster_os1_32.dae" />
+          <mesh filename="package://ros_components_description/meshes/ouster_os1_32.dae" />
         </geometry>
       </visual>

File: urdf/slamtec_rplidar_a2.urdf.xacro (robot description, xacro)
@@ -64,5 +64,5 @@
         <origin xyz="0.0 0.0 0.0" rpy="0.0 0.0 0.0" />
         <geometry>
-          <mesh filename="file://$(find ros_components_description)/meshes/${mesh}" />
+          <mesh filename="package://ros_components_description/meshes/${mesh}" />
         </geometry>
       </visual>

File: urdf/slamtec_rplidar_a3.urdf.xacro (robot description, xacro)
@@ -42,5 +42,5 @@
         <geometry>
           <!-- slamtec_rplidar_ax.dae is used as a shared mesh for A2 and A3 rplidars -->
-          <mesh filename="file://$(find ros_components_description)/meshes/slamtec_rplidar_ax.dae" />
+          <mesh filename="package://ros_components_description/meshes/slamtec_rplidar_ax.dae" />
         </geometry>
       </visual>

File: urdf/slamtec_rplidar_s1.urdf.xacro (robot description, xacro)
@@ -41,5 +41,5 @@
         <origin xyz="0.0 0.0 0.0" rpy="0.0 0.0 0.0" />
         <geometry>
-          <mesh filename="file://$(find ros_components_description)/meshes/slamtec_rplidar_s1.dae" />
+          <mesh filename="package://ros_components_description/meshes/slamtec_rplidar_s1.dae" />
         </geometry>
       </visual>

File: urdf/velodyne_puck.urdf.xacro (robot description, xacro)
@@ -31,5 +31,5 @@
         <origin xyz="0.0 0.0 0.0" rpy="0.0 0.0 0.0" />
         <geometry>
-          <mesh filename="file://$(find ros_components_description)/meshes/velodyne_puck.dae" />
+          <mesh filename="package://ros_components_description/meshes/velodyne_puck.dae" />
         </geometry>
       </visual>
